File: pcb/Seed3-DevKit-Eurorack-Rev1/Seed3-DevKit-Eurorack_2.kicad_sch (KiCad schematic)
At the start: 48 parts, among them Q1 MMBT3904, Q2 MMBT3904, SW1 TOGGLE_ON_OFF_ON_PIP2, SW2 TOGGLE_ON-ON_PIP3, SW3 PTH Mini Button, SW4 PTH Mini Button, U11 H11L1, U7 MICRO_SD_CARD

Commit message: finished routing board, fixed DRCs, and added cutout to PCB.
Parts:
- SW1: footprint parts-for-kicad:TOGGLE_SILK_PIP3 -> parts-for-kicad:TOGGLE_ON_OFF_ON_SILK
- SW2: footprint parts-for-kicad:TOGGLE_SILK_PIP3 -> parts-for-kicad:TOGGLE_ON-ON_SILK
- VR1, VR2, VR3, VR4, VR5, VR6, VR7, VR8: footprint parts-for-kicad:9MM_SNAP-IN_POT_SILK_PIP -> parts-for-kicad:9MM_SNAP-IN_POT_SILK
Changed lines of the file:
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@@
 			)
 		)
-		(property "Footprint" "parts-for-kicad:TOGGLE_SILK_PIP3"
+		(property "Footprint" "parts-for-kicad:TOGGLE_ON_OFF_ON_SILK"
 			(at 88.9 80.01 0)
 			(effects
@@
 			)
 		)
-		(property "Footprint" "parts-for-kicad:9MM_SNAP-IN_POT_SILK_PIP"
+		(property "Footprint" "parts-for-kicad:9MM_SNAP-IN_POT_SILK"
 			(at 199.39 45.72 0)
 			(effects
@@
 			)
 		)
-		(property "Footprint" "parts-for-kicad:9MM_SNAP-IN_POT_SILK_PIP"
+		(property "Footprint" "parts-for-kicad:9MM_SNAP-IN_POT_SILK"
 			(at 124.46 45.72 0)
 			(effects
@@
 			)
 		)
-		(property "Footprint" "parts-for-kicad:TOGGLE_SILK_PIP3"
+		(property "Footprint" "parts-for-kicad:TOGGLE_ON-ON_SILK"
 			(at 50.8 80.01 0)
 			(effects
@@
 			)
 		)
-		(property "Footprint" "parts-for-kicad:9MM_SNAP-IN_POT_SILK_PIP"
+		(property "Footprint" "parts-for-kicad:9MM_SNAP-IN_POT_SILK"
 			(at 105.41 45.72 0)
 			(effects
@@
 			)
 		)
-		(property "Footprint" "parts-for-kicad:9MM_SNAP-IN_POT_SILK_PIP"
+		(property "Footprint" "parts-for-kicad:9MM_SNAP-IN_POT_SILK"
 			(at 142.24 45.72 0)
 			(effects
@@
 			)
 		)
-		(property "Footprint" "parts-for-kicad:9MM_SNAP-IN_POT_SILK_PIP"
+		(property "Footprint" "parts-for-kicad:9MM_SNAP-IN_POT_SILK"
 			(at 85.09 45.72 0)
 			(effects
@@
 			)
 		)
-		(property "Footprint" "parts-for-kicad:9MM_SNAP-IN_POT_SILK_PIP"
+		(property "Footprint" "parts-for-kicad:9MM_SNAP-IN_POT_SILK"
 			(at 180.34 45.72 0)
 			(effects
@@
 			)
 		)
-		(property "Footprint" "parts-for-kicad:9MM_SNAP-IN_POT_SILK_PIP"
+		(property "Footprint" "parts-for-kicad:9MM_SNAP-IN_POT_SILK"
 			(at 161.29 45.72 0)
 			(effects
@@
 			)
 		)
-		(property "Footprint" "parts-for-kicad:9MM_SNAP-IN_POT_SILK_PIP"
+		(property "Footprint" "parts-for-kicad:9MM_SNAP-IN_POT_SILK"
 			(at 62.23 45.72 0)
 			(effects
